Commit message: refactor:Rebuild model using macros

File: models/urdf/delivery_robot.xacro (robot description, xacro)
@@ -12,4 +12,6 @@
   <xacro:property name="caster_radius" value="${(wheel_radius-base_chassis_height/4)/2}"/>
   <xacro:property name="caster_mass" value="0.1"/>
+  <!-- Include gazebo properties -->
+  <xacro:include filename="$(find delivery_robot_simulation)/models/urdf/delivery_robot.gazebo" />
   <!-- Define inertia macros  -->
   <xacro:macro name="cuboid_inertia" params="m x y z">
@@ -36,5 +38,5 @@
         </geometry>
       </collision>
-      <visual name='right_wheel_visual'>
+      <visual name='${position_name}_wheel_visual'>
         <origin xyz="0.0 0 0" rpy=" 0 1.5707 1.5707"/>
         <geometry>
@@ -65,5 +67,5 @@
         </geometry>
       </collision>
-      <visual name='right_caster_visual'>
+      <visual name='${position_name}_caster_visual'>
         <origin xyz="0 0 0" rpy=" 0 0 0"/>
         <geometry>
@@ -80,7 +82,34 @@
     </joint>
   </xacro:macro>
+  <!-- Define a container wall macro -->
+  <xacro:macro name="container_wall" params="wall_name wall_mass wall_thick wall_height is_y is_x direction_x_factor direction_y_factor">
+    <link name='${wall_name}_container_side'>
+      <pose>0 0 0 0 0 0</pose>
+      <inertial>
+        <mass value="${wall_mass}"/>
+        <origin xyz="0 0 0" rpy=" 0 0 0"/>
+        <xacro:cuboid_inertia m="${wall_mass}" x="${is_y*wall_thick + is_x*base_chassis_length}" y="${is_x*wall_thick + is_y*base_chassis_width}" z="${wall_height}" />
+      </inertial>
+      <collision name='collision'>
+        <origin xyz="0 0 0" rpy=" 0 0 0"/>
+        <geometry>
+          <box size="${is_y*wall_thick + is_x*base_chassis_length} ${is_x*wall_thick + is_y*base_chassis_width} ${wall_height}"/>
+        </geometry>
+      </collision>
+      <visual name='base_chassis_visual'>
+        <origin xyz="0 0 0" rpy=" 0 0 0"/>
+        <geometry>
+          <box size="${is_y*wall_thick + is_x*base_chassis_length} ${is_x*wall_thick + is_y*base_chassis_width} ${wall_height}"/>
+        </geometry>
+      </visual>
+    </link>
+    <joint type="fixed" name="${wall_name}_container_side_hinge">
+      <origin xyz="${direction_x_factor*((base_chassis_length - wall_thick)/2)} ${direction_y_factor*((base_chassis_width - wall_thick)/2)} ${((base_chassis_height+wall_height)/2)}" rpy="0 0 0"/>
+      <child link="${wall_name}_container_side"/>
+      <parent link="base_chassis"/>
+    </joint>
+  </xacro:macro>
+  <!-- Robot definitions -->
   <link name="robot_footprint"></link>
-  <!-- Include gazebo properties -->
-  <xacro:include filename="$(find delivery_robot_simulation)/models/urdf/delivery_robot.gazebo" />
   <joint name="robot_footprint_joint" type="fixed">
     <origin xyz="0 0 0" rpy="0 0 0" />
@@ -89,5 +118,5 @@
   </joint>
   <link name='base_chassis'>
-    <pose>0 0 0.12 0 0 0</pose>
+    <pose>0 0 0 0 0 0</pose>
     <inertial>
       <mass value="${base_chassis_mass}"/>
@@ -101,5 +130,5 @@
       </geometry>
     </collision>
-    <visual name='chassis_visual'>
+    <visual name='base_chassis_visual'>
       <origin xyz="0 0 0" rpy=" 0 0 0"/>
       <geometry>
@@ -108,38 +137,17 @@
     </visual>
   </link>
-  <!-- ### WHEELS ### -->
+  <!-- Wheels definitions -->
   <xacro:wheel position_name="left" direction_factor="1"/>
   <xacro:wheel position_name="right" direction_factor="-1"/>
-  <!-- Ball caster definitions -->
+  <!-- Ball casters definitions -->
   <xacro:ball_caster position_name="front_left" direction_x_factor="1" direction_y_factor="1"/>
   <xacro:ball_caster position_name="front_right" direction_x_factor="1" direction_y_factor="-1"/>
   <xacro:ball_caster position_name="back_left" direction_x_factor="-1" direction_y_factor="1"/>
   <xacro:ball_caster position_name="back_right" direction_x_factor="-1" direction_y_factor="-1"/>
-  <!--
-  <link name='base_hokuyo'>
-    <inertial>
-      <mass value="0.01"/>
-      <origin xyz="0 0 0" rpy=" 0 0 0"/>
-      <inertia ixx="0.000016667" ixy = "0" ixz = "0" iyy="0.00004167" iyz = "0" izz="0.00004167" />
-    </inertial>
-    <collision name='collision'>
-      <origin xyz="0 0 0" rpy=" 0 0 0"/>
-      <geometry>
-        <box size="0.2 0.1 0.1"/>
-      </geometry>
-    </collision>
-    <visual name='sup_visual'>
-      <origin xyz="0 0 0" rpy=" 0 0 0"/>
-      <geometry>
-        <box size="0.2 0.1 0.1"/>
-      </geometry>
-    </visual>
-  </link>
-  <joint type="fixed" name="base_hokuyo_joint">
-    <origin xyz="0 0 0.12" rpy="0 0 0"/>
-    <child link="base_hokuyo"/>
-    <parent link="base_chassis"/>
-  </joint>
--->
+  <!-- Container definitions -->
+  <xacro:container_wall wall_name="left" wall_mass="0.01" wall_thick="0.01" wall_height="0.1" is_y="0" is_x="1" direction_x_factor="0" direction_y_factor="1" />
+  <xacro:container_wall wall_name="right" wall_mass="0.01" wall_thick="0.01" wall_height="0.1" is_y="0" is_x="1" direction_x_factor="0" direction_y_factor="-1" />
+  <xacro:container_wall wall_name="front" wall_mass="0.01" wall_thick="0.1" wall_height="0.1" is_y="1" is_x="0" direction_x_factor="1" direction_y_factor="0" />
+  <xacro:container_wall wall_name="back" wall_mass="0.01" wall_thick="0.01" wall_height="0.1" is_y="1" is_x="0" direction_x_factor="-1" direction_y_factor="0" />
   <!-- ### CAMERA ### -->
   <link name="camera_link">
@@ -148,5 +156,4 @@
       <origin xyz="0.0 0 0" rpy=" 0 0 0"/>
       <xacro:cuboid_inertia m="0.1" x="0.05" y="0.05" z="0.05" />
-      <!-- <inertia ixx="1e-6" ixy="0" ixz="0" iyy="1e-6" iyz="0" izz="1e-6" /> -->
     </inertial>
     <collision name='camera_collision'>
@@ -156,5 +163,5 @@
       </geometry>
     </collision>
-    <visual name='camera_visual'>
+    <visual name='camera_link_visual'>
       <origin xyz="0 0 0" rpy=" 0 0 0"/>
       <geometry>
@@ -166,5 +173,5 @@
   </link>
   <joint type="fixed" name="camera_joint">
-    <origin xyz="${base_chassis_length/2+0.025} 0 0.075" rpy="0 0 0"/>
+    <origin xyz="${base_chassis_length/2+0.025} 0 ${base_chassis_height/2-0.025}" rpy="0 0 0"/>
     <child link="camera_link"/>
     <parent link="base_chassis"/>
@@ -182,5 +189,4 @@
       <origin xyz="0.0 0 0" rpy=" 0 0 0"/>
       <xacro:cuboid_inertia m="0.00001" x="0.1" y="0.1" z="0.1" />
-      <!-- <inertia ixx="1e-6" ixy="0" ixz="0" iyy="1e-6" iyz="0" izz="1e-6" /> -->
     </inertial>
     <collision name='hokuyo_collision'>
@@ -198,5 +204,5 @@
   </link>
   <joint type="fixed" name="hokuyo_joint">
-    <origin xyz="${base_chassis_length/2-0.05} 0 ${base_chassis_height/2+0.05}" rpy="0 0 0"/>
+    <origin xyz="${base_chassis_length/2-0.05} 0 ${base_chassis_height/2+0.05+0.1}" rpy="0 0 0"/>
     <child link="hokuyo"/>
     <parent link="base_chassis"/>

Commit message: chore: Adjust simulation package name

File: models/urdf/delivery_robot.xacro (robot description, xacro)
@@ -13,5 +13,5 @@
   <xacro:property name="caster_mass" value="0.1"/>
   <!-- Include gazebo properties -->
-  <xacro:include filename="$(find delivery_robot_simulation)/models/urdf/delivery_robot.gazebo" />
+  <xacro:include filename="$(find warehouse_robot_simulation)/models/urdf/delivery_robot.gazebo" />
   <!-- Define inertia macros  -->
   <xacro:macro name="cuboid_inertia" params="m x y z">
@@ -199,5 +199,5 @@
       <origin xyz="0 0 0" rpy=" 0 0 0"/>
       <geometry>
-        <mesh filename="package://delivery_robot_simulation/models/meshes/hokuyo.dae"/>
+        <mesh filename="package://warehouse_robot_simulation/models/meshes/hokuyo.dae"/>
       </geometry>
     </visual>
